File: LedTree_hw/LedTree.sch (KiCad schematic (older format))
At the start: 97 parts, among them U1 USBLC6

Commit message: + PCB is ready
Parts:
- removed HOLE1, HOLE2, HOLE3, HOLE4: HOLE_METALLED, PCB:Hole3_5_out6mm, symbol pcb_details:HOLE_METALLED
- removed Logo1: Logo, Pictures:Ostranna_16d9_13d5, symbol pcb_details:Logo
- removed R14: 0R15, Resistors:RES_1206, symbol Tittar_kl:R
- removed TP7: TESTPOINT, PCB:TESTPOINT_1MM, symbol pcb_details:TESTPOINT
- removed XL8: USB_MICRO, Connectors:USBmicro_MOLEX_1050170001, symbol Connectors_kl:USB_MICRO_4H
- added C37, C38, C39: 0.1u, Capacitors:CAP_0603, symbol Tittar_kl:C
- added D2, D3: PESD3V3, Diodes:SOD323, symbol Tittar_kl:ZenerBidir
- added R10, R11, R15, R16, R17, R18, R21, R22, R23, R24, R26, R27, R28, R29, R5, R7: 0R56, Resistors:RES_0805, symbol Tittar_kl:R
- added R33: 100k, Resistors:RES_0603, symbol Tittar_kl:R
- added R34, R35, R36, R37: 10k, Resistors:RES_0603, symbol Tittar_kl:R
- added XL11: CONN_2, Connectors:W02_Pitch_2d54, symbol Connectors_kl:CONN_2
- added XL12, XL13: CONN_2, Connectors:XY122V-2, symbol Connectors_kl:CONN_2
- added XL14: CONN_4, Connectors:WB-04(MW-4M), symbol Connectors_kl:CONN_4
- added XL8: USB_B, Connectors:USB_B_Vertical_1JF, symbol Connectors_kl:USB_A
- C31: footprint Capacitors:CAP_0805 -> Capacitors:CAP_0603_Silks
- C32: footprint Capacitors:CAP_0805 -> Capacitors:CAP_0603_Silks; PN GRM21BR61C106KE15L -> (none)
- C36: footprint Capacitors:CAP_10Rx16_HOR -> Capacitors:CAP_10xxR
- R12, R4, R6, R9: value 0R15 -> 0R56; footprint Resistors:RES_1206 -> Resistors:RES_0805
- XL10: footprint Connectors:2ZHDRC-02P -> Connectors:XY122V-2
- XL2, XL3, XL4, XL5, XL7: footprint PCB:Oval3x1.5wHole0d9_x2 -> Connectors:XY122V-2
- XL6: footprint (none) -> Connectors:WB-03(MW-3M)
- renumbered D2 to D4, R7 to R13, R8 to R14, R10 to R19, R11 to R20, R13 to R25, R15 to R30, R16 to R31, R17 to R32, R5 to R8, TP9 to TP10, TP10 to TP6, TP6 to TP7, TP8 to TP9
Connections:
- net +3v3: now also C37.2, R34.1, R35.1, XL14.2 (PM)
- net 5V_USB: now also XL8.1 (UVcc)
- net DIN+: now also U1.1 (I/O1), XL8.3 (D+); no longer U1.3 (I/O2)
- net DIN-: now also U1.3 (I/O2), XL8.2 (D-); no longer U1.1 (I/O1)
- net GND: now also C37.1, C38.1, C39.1, D2.A, D3.A, R33.2, XL14.1 (P1); no longer C29.2, U1.2 (GND)
- net GNDPWR: now also C29.2, U1.2 (GND), R10.2, R11.2, R15.2, R16.2, R17.2, R18.2, R21.2, R22.2, R23.2, R24.2, R26.2, R27.2, R28.2, R29.2, R5.2, R7.2, XL8.4 (UGND)
- net USB_D+: now also U1.6 (I/O1); no longer U1.4 (I/O2)
- net USB_D-: now also U1.4 (I/O2); no longer U1.6 (I/O1)
- net VDDA: now also D2.C
- net NL7: now reaches DA6.7 (SW), L7.2
- net NL1: now reaches DA1.1 (SW), L1.2
- net FB1: now reaches DA1.5 (FB), R4.1, XL2.2 (PM)
- net FB1: now also R6.1, R5.1, R7.1
- net ENC_A: now reaches DD1.14 (ADC12-5/WKUP1/T2C1/T5C1/TX4/PA0)
- net ENC_A: now also C38.2, R36.1
- net ENC_B: now reaches DD1.15 (ADC12-6/T2C2/T5C2/RX4/PA1)
- net ENC_B: now also C39.2, R37.1
- net LD1: now reaches C1.1, L1.1, XL2.1 (P1)
- net LD2: now reaches C4.1, L2.1, XL3.1 (P1)
- net FB2: now reaches DA2.5 (FB), XL3.2 (PM)
- net FB2: now also R12.1, R9.1, R10.1, R11.1; no longer R6.1
- net NL2: now reaches DA2.1 (SW), L2.2
- net LD4: now reaches C14.1, L5.1, XL5.1 (P1)
- net FB4: now reaches DA4.5 (FB), XL5.2 (PM)
- net FB4: now also R21.1, R22.1, R23.1, R24.1; no longer R12.1
- net NL4: now reaches DA4.1 (SW), L5.2
- net LD3: now reaches C9.1, L3.1, XL4.1 (P1)
- net FB3: now reaches DA3.5 (FB), XL4.2 (PM)
- net FB3: now also R15.1, R16.1, R17.1, R18.1; no longer R9.1
- net NL3: now reaches DA3.1 (SW), L3.2
- net LD5: now reaches C26.1, L6.1, XL7.1 (P1)
- net FB5: now reaches DA5.5 (FB), XL7.2 (PM)
- net FB5: now also R26.1, R27.1, R28.1, R29.1
- net NL5: now reaches DA5.1 (SW), L6.2
- net at R19.1, XL6.2 (PM): now also D3.C, R33.1
- new net: R35.2, R37.2, XL14.3
- new net: R34.2, R36.2, XL14.4
- new net HV1: XL11.1 (P1), XL12.1 (P1)
- new net HV2: XL11.2 (PM), XL13.1 (P1)
- new net HV3: XL12.2 (PM), XL13.2 (PM)
- no-connect marks 41 -> 36
Other:
- note added: "220v in"
- note added: "220v out"
- note added: "220v switch"
- note added: "Encoder"
- note added: "RVar switch"
- moved on the sheet: C12, C13, C17, C18, C19, C20, C21, C22, C23, C24, C25, C5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
